Commit message: Isaac ROS 4.1

File: isaac_manipulator_robot_description/urdf/ur10e_robotiq_base_sim.ros2_control.xacro (robot description, xacro)
@@ -42,6 +42,6 @@
       <joint name="elbow_joint">
         <command_interface name="position">
-          <param name="min">{-pi}</param>
-          <param name="max">{pi}</param>
+          <param name="min">-3.14159</param>
+          <param name="max">3.14159</param>
         </command_interface>
         <command_interface name="velocity">

File: isaac_manipulator_robot_description/urdf/ur_robotiq_gripper.urdf.xacro (robot description, xacro)
@@ -2,5 +2,5 @@
 <robot xmlns:xacro="http://wiki.ros.org/xacro" name="robotiq_gripper">
     <!-- parameters -->
-    <xacro:arg name="use_fake_hardware" default="false" />
+    <xacro:arg name="use_mock_hardware" default="false" />
     <xacro:arg name="com_port" default="/tmp/ttyUR" />
     <xacro:arg name="gripper_speed" default="0.150" /> <!-- unknown -->
@@ -27,5 +27,5 @@
         prefix=""
         parent="tool0"
-        use_fake_hardware="$(arg use_fake_hardware)"
+        use_fake_hardware="$(arg use_mock_hardware)"
         com_port="$(arg com_port)"
         sim_isaac="$(arg sim_isaac)"

File: isaac_manipulator_robot_description/urdf/ur_sim.urdf.xacro (robot description, xacro)
@@ -41,7 +41,9 @@
    <xacro:arg name="tool_device_name" default="/tmp/ttyUR" />
    <xacro:arg name="tool_tcp_port" default="54321" />
-     <!-- Simulation parameters -->
+   <!-- Simulation parameters -->
    <xacro:arg name="use_fake_hardware" default="false" />
    <xacro:arg name="fake_sensor_commands" default="false" />
+   <xacro:arg name="use_mock_hardware" default="$(arg use_fake_hardware)" />
+   <xacro:arg name="mock_sensor_commands" default="$(arg fake_sensor_commands)" />
    <xacro:arg name="sim_gazebo" default="false" />
    <xacro:arg name="sim_ignition" default="false" />
@@ -68,4 +70,6 @@
      use_fake_hardware="$(arg use_fake_hardware)"
      fake_sensor_commands="$(arg fake_sensor_commands)"
+     use_mock_hardware="$(arg use_mock_hardware)"
+     mock_sensor_commands="$(arg mock_sensor_commands)"
      sim_gazebo="$(arg sim_gazebo)"
      sim_ignition="$(arg sim_ignition)"

File: isaac_manipulator_robot_description/urdf/ur_sim_macro.xacro (robot description, xacro)
@@ -60,4 +60,6 @@
     use_fake_hardware:=false
     fake_sensor_commands:=false
+    use_mock_hardware:=false
+    mock_sensor_commands:=false
     sim_gazebo:=false
     sim_ignition:=false
@@ -98,7 +100,7 @@
       <xacro:ur_ros2_control
         name="${name}"
-        use_fake_hardware="${use_fake_hardware}"
+        use_mock_hardware="${use_mock_hardware}"
         initial_positions="${initial_positions}"
-        fake_sensor_commands="${fake_sensor_commands}"
+        mock_sensor_commands="${mock_sensor_commands}"
         headless_mode="${headless_mode}"
         sim_gazebo="${sim_gazebo}"
@@ -135,5 +137,5 @@
     <link name="${tf_prefix}base_link_inertia">
       <visual>
-        <origin xyz="0 0 0" rpy="0 0 ${pi}"/>
+        <origin xyz="0 0 0" rpy="0 0 3.14159"/>
         <geometry>
           <xacro:get_mesh name="base" type="visual"/>
@@ -141,5 +143,5 @@
       </visual>
       <collision>
-        <origin xyz="0 0 0" rpy="0 0 ${pi}"/>
+        <origin xyz="0 0 0" rpy="0 0 3.14159"/>
         <geometry>
           <xacro:get_mesh name="base" type="collision"/>
@@ -152,5 +154,5 @@
     <link name="${tf_prefix}shoulder_link">
       <visual>
-        <origin xyz="0 0 0" rpy="0 0 ${pi}"/>
+        <origin xyz="0 0 0" rpy="0 0 3.14159"/>
         <geometry>
           <xacro:get_mesh name="shoulder" type="visual"/>
@@ -158,5 +160,5 @@
       </visual>
       <collision>
-        <origin xyz="0 0 0" rpy="0 0 ${pi}"/>
+        <origin xyz="0 0 0" rpy="0 0 3.14159"/>
         <geometry>
           <xacro:get_mesh name="shoulder" type="collision"/>
@@ -329,5 +331,5 @@
            link/frame) to introduce the necessary rotation over Z (of pi rad).
       -->
-      <origin xyz="0 0 0" rpy="0 0 ${pi}" />
+      <origin xyz="0 0 0" rpy="0 0 3.14159" />
     </joint>
     <joint name="${tf_prefix}shoulder_pan_joint" type="revolute">
@@ -415,5 +417,5 @@
       <parent link="${tf_prefix}wrist_3_link"/>
       <child link="${tf_prefix}ft_frame"/>
-      <origin xyz="0 0 0" rpy="${pi} 0 0"/>
+      <origin xyz="0 0 0" rpy="3.14159 0 0"/>
     </joint>
     <!-- ROS-Industrial 'base' frame - base_link to UR 'Base' Coordinates transform -->
@@ -425,5 +427,5 @@
            the UR controller.
       -->
-      <origin xyz="0 0 0" rpy="0 0 ${pi}"/>
+      <origin xyz="0 0 0" rpy="0 0 3.14159"/>
       <parent link="${tf_prefix}base_link"/>
       <child link="${tf_prefix}base"/>
